File: Micro T_Probe.sch (KiCad schematic (older format))
At the start: 11 parts, among them P1 CONN_5, P2 CONN_5, U1 TMP_102

Commit message: Updated the solderability of this board by removing the mask above the solder junctions and enlarging the pads.
Parts:
- GS1: value GS2 -> 00
- GS2: value GS2 -> 01
- GS3: value GS2 -> 11
- GS4: value GS2 -> 10
Changed lines of the file:
@@
 Sheet 1 1
 Title ""
-Date "24 jul 2013"
+Date "3 aug 2014"
 Rev ""
 Comp ""
@@
 P 5850 2150
 F 0 "GS1" H 5950 2300 50  0000 C CNN
-F 1 "GS2" H 5950 2001 40  0000 C CNN
+F 1 "00" H 5950 2001 40  0000 C CNN
 F 2 "" H 5850 2150 60  0000 C CNN
 F 3 "" H 5850 2150 60  0000 C CNN
@@
 P 5850 2400
 F 0 "GS3" H 5950 2550 50  0000 C CNN
-F 1 "GS2" H 5950 2251 40  0000 C CNN
+F 1 "11" H 5950 2251 40  0000 C CNN
 F 2 "" H 5850 2400 60  0000 C CNN
 F 3 "" H 5850 2400 60  0000 C CNN
@@
 P 5850 2650
 F 0 "GS4" H 5950 2800 50  0000 C CNN
-F 1 "GS2" H 5950 2501 40  0000 C CNN
+F 1 "10" H 5950 2501 40  0000 C CNN
 F 2 "" H 5850 2650 60  0000 C CNN
 F 3 "" H 5850 2650 60  0000 C CNN
@@
 P 5850 2900
 F 0 "GS2" H 5950 3050 50  0000 C CNN
-F 1 "GS2" H 5950 2751 40  0000 C CNN
+F 1 "01" H 5950 2751 40  0000 C CNN
 F 2 "" H 5850 2900 60  0000 C CNN
 F 3 "" H 5850 2900 60  0000 C CNN
